File: Vision.sch (KiCad schematic (older format))
At the start: 191 parts, among them Q1 2N7002, SW2 SW_Push, SW3 SW_SPDT, U2 PRTR5V0U2X, U3 STM32F072CBUx, U4 MCP1700-3002E_SOT23

Commit message: Update schematics
Parts:
- removed C1, C10, C11, C13, C14, C15, C16, C17, C18, C9: 0.1uF, Capacitors_SMD:C_0603, symbol Device:C_Small
- removed D42, D44, D63, D64: SOD-123, Diodes_SMD:D_SOD-123, symbol Device:D_Small
- removed K_CAPS2: MX-1.25U, MX_Alps_Hybrid:MX-1.25U-FLIPPED, symbol MX_Alps_Hybrids:MX-1U
- removed K_ENTER1: MX-2.25U, MX_Alps_Hybrid:MX-2.25U, symbol MX_Alps_Hybrids:MX-1U
- removed K_ENTER2, K_RCTRL1, K_SHIFT2: MX-1.25U, MX_Alps_Hybrid:MX-1.25U, symbol MX_Alps_Hybrids:MX-1U
- removed K_ENTER3: MX-ISO, MX_Alps_Hybrid:MX-ISO-ReversedStabilizers, symbol MX_Alps_Hybrids:MX-1U
- removed K_LSPACE2: MX-2.75U, MX_Alps_Hybrid:MX-2.75U-FLIPPED-ReversedStabilizers, symbol MX_Alps_Hybrids:MX-1U
- removed K_RSHIFT2: MX-1.75U, MX_Alps_Hybrid:MX-1.75U, symbol MX_Alps_Hybrids:MX-1U
- removed K_RSHIFT3, K_SHIFT3, K_SPACE3: MX-1U, MX_Alps_Hybrid:MX-1U, symbol MX_Alps_Hybrids:MX-1U
- removed K_RSHIFT4: MX-2.75U, MX_Alps_Hybrid:MX-2.75U, symbol MX_Alps_Hybrids:MX-1U
- removed K_RSPACE2: MX-2.25U, MX_Alps_Hybrid:MX-2.25U-FLIPPED-ReversedStabilizers, symbol MX_Alps_Hybrids:MX-1U
- removed K_RWIN1: MX-1.25U, MX_Alps_Hybrid:MX-1U, symbol MX_Alps_Hybrids:MX-1U
- removed K_SPACE4: MX-1U, MX_Alps_Hybrid:MX-1U-FLIPPED, symbol MX_Alps_Hybrids:MX-1U
- removed K_\1: MX-1.5U, MX_Alps_Hybrid:MX-1.5U, symbol MX_Alps_Hybrids:MX-1U
- removed Q1: 2N7002, TO_SOT_Packages_SMD:SOT-23, symbol Transistor_FET:2N7002
- removed R16, R17, R18, R19, R20, R21, R22, R23, R24, R25, R26, R27, R31, R32, R33, R34, R35, R36, R37, R38, R39, R40, R41, R42, R44, R45, R46, R47, R48, R49, R50, R51, R52, R53, R54, R55, R58, R59, R60, R61, R62, R63, R64, R72: 1k, Resistors_SMD:R_0805, symbol Device:R_Small
- removed R3: 5.1k, Resistors_SMD:R_0805, symbol Device:R_Small
- removed R69: 100, Resistors_SMD:R_0805, symbol Device:R_Small
- removed RGB1, RGB10, RGB11, RGB12, RGB2, RGB3, RGB4, RGB5, RGB6, RGB7, RGB8, RGB9: WS2812B, LEDs:LED_WS2812B-PLCC4, symbol LED:WS2812B
- removed SW3: SW_SPDT, Buttons_Switches_SMD:SW_SPDT_PCM12, symbol Switch:SW_SPDT
- removed U2: PRTR5V0U2X, random-keyboard-parts:SOT143B, symbol ai03-locallib:PRTR5V0U2X
- added C3: 4.7nF, Capacitor_SMD:C_0603_1608Metric, symbol Device:C_Small
- added C4: 10uF, Capacitor_SMD:C_0603_1608Metric, symbol Device:C_Small
- added D1, D14, D15, D27, D34, D40, D48: SOD-123, Diode_SMD:D_SOD-123, symbol Device:D_Small
- added D49: BAT41ZFILM, Diode_SMD:D_SOD-123, symbol Device:D_Schottky_Small
- added D50: SMF9.0CA, Diode_SMD:D_SOD-123, symbol Device:D_TVS
- added D51: 1N4148W, Diode_SMD:D_SOD-123, symbol Diode:1N4148
- added J1: Conn_ARM_JTAG_SWD_10, Connector_PinHeader_2.54mm:PinHeader_2x05_P2.54mm_Vertical, symbol Connector:Conn_ARM_JTAG_SWD_10
- added K_B2, K_P2: MX-1U, MX_Only:MXOnly-1U-Hotswap-Antishear, symbol MX_Alps_Hybrid:MX-NoLED
- added K_CTRL2: MX-1.25U, MX_Only:MXOnly-1U-Hotswap-Antishear, symbol MX_Alps_Hybrid:MX-NoLED
- added K_DEL1, K_PGUP1: MX-1.5U, MX_Only:MXOnly-1U-Hotswap-Antishear, symbol MX_Alps_Hybrid:MX-NoLED
- added K_ENTER1: MX-2.25U, MX_Only:MXOnly-1U-Hotswap-Antishear, symbol MX_Alps_Hybrid:MX-NoLED
- added K_FN1, K_PGDN1: MX-1.75U, MX_Only:MXOnly-1U-Hotswap-Antishear, symbol MX_Alps_Hybrid:MX-NoLED
- added Q1: DTC123J, Package_TO_SOT_SMD:SC-59, symbol Transistor_BJT:DTC123J
- added R4: 1M, Resistors_SMD:R_0805, symbol Device:R_Small
- added R6: 100k, Resistors_SMD:R_0805, symbol Device:R_Small
- added U3: TPD4E05U06DQAR, random-keyboard-parts:USON-TPDxE05U06, symbol random-keyboard-parts:TPD4E05U06DQAR
- C1: renamed from C25; footprint Capacitors_SMD:C_0603 -> Capacitor_SMD:C_0603_1608Metric
- C10: renamed from C23; value 4.7uF -> 1uF; footprint Capacitors_SMD:C_0603 -> Capacitor_SMD:C_0603_1608Metric
- C11: renamed from C24; footprint Capacitors_SMD:C_0603 -> Capacitor_SMD:C_0603_1608Metric
- C12, C5: value 0.1uF -> 4.7uF; footprint Capacitors_SMD:C_0603 -> Capacitor_SMD:C_0603_1608Metric
- C2: renamed from C26; footprint Capacitors_SMD:C_0603 -> Capacitor_SMD:C_0603_1608Metric
- C6: renamed from C19; value 0.1uF -> 10nF; footprint Capacitors_SMD:C_0603 -> Capacitor_SMD:C_0603_1608Metric
- C7: renamed from C20; value 0.1uF -> 100nF; footprint Capacitors_SMD:C_0603 -> Capacitor_SMD:C_0603_1608Metric
- C8: renamed from C21; value 0.1uF -> 100nF; footprint Capacitors_SMD:C_0603 -> Capacitor_SMD:C_0603_1608Metric
- C9: renamed from C22; value 0.1uF -> 100nF; footprint Capacitors_SMD:C_0603 -> Capacitor_SMD:C_0603_1608Metric
- D10: renamed from D24; footprint Diodes_SMD:D_SOD-123 -> Diode_SMD:D_SOD-123
- D11: renamed from D25; footprint Diodes_SMD:D_SOD-123 -> Diode_SMD:D_SOD-123
- D12: renamed from D26; footprint Diodes_SMD:D_SOD-123 -> Diode_SMD:D_SOD-123
- D13: renamed from D27; footprint Diodes_SMD:D_SOD-123 -> Diode_SMD:D_SOD-123
- D16: renamed from D31; footprint Diodes_SMD:D_SOD-123 -> Diode_SMD:D_SOD-123
- D17: renamed from D32; footprint Diodes_SMD:D_SOD-123 -> Diode_SMD:D_SOD-123
- D18: renamed from D33; footprint Diodes_SMD:D_SOD-123 -> Diode_SMD:D_SOD-123
- D19: renamed from D34; footprint Diodes_SMD:D_SOD-123 -> Diode_SMD:D_SOD-123
- D2: renamed from D16; footprint Diodes_SMD:D_SOD-123 -> Diode_SMD:D_SOD-123
- D20: renamed from D35; footprint Diodes_SMD:D_SOD-123 -> Diode_SMD:D_SOD-123
- D21: renamed from D36; footprint Diodes_SMD:D_SOD-123 -> Diode_SMD:D_SOD-123
- D22: renamed from D37; footprint Diodes_SMD:D_SOD-123 -> Diode_SMD:D_SOD-123
- D23: renamed from D38; footprint Diodes_SMD:D_SOD-123 -> Diode_SMD:D_SOD-123
- D24: renamed from D39; footprint Diodes_SMD:D_SOD-123 -> Diode_SMD:D_SOD-123
- D25: renamed from D40; footprint Diodes_SMD:D_SOD-123 -> Diode_SMD:D_SOD-123
- D26: renamed from D41; footprint Diodes_SMD:D_SOD-123 -> Diode_SMD:D_SOD-123
- D28: renamed from D45; footprint Diodes_SMD:D_SOD-123 -> Diode_SMD:D_SOD-123
- D29: renamed from D46; footprint Diodes_SMD:D_SOD-123 -> Diode_SMD:D_SOD-123
- D3: renamed from D17; footprint Diodes_SMD:D_SOD-123 -> Diode_SMD:D_SOD-123
- D30: renamed from D47; footprint Diodes_SMD:D_SOD-123 -> Diode_SMD:D_SOD-123
- D31: renamed from D48; footprint Diodes_SMD:D_SOD-123 -> Diode_SMD:D_SOD-123
- D32: renamed from D49; footprint Diodes_SMD:D_SOD-123 -> Diode_SMD:D_SOD-123
- D33: renamed from D50; footprint Diodes_SMD:D_SOD-123 -> Diode_SMD:D_SOD-123
- D35: renamed from D51; footprint Diodes_SMD:D_SOD-123 -> Diode_SMD:D_SOD-123
- D36: renamed from D52; footprint Diodes_SMD:D_SOD-123 -> Diode_SMD:D_SOD-123
- D37: renamed from D53; footprint Diodes_SMD:D_SOD-123 -> Diode_SMD:D_SOD-123
- D38: renamed from D54; footprint Diodes_SMD:D_SOD-123 -> Diode_SMD:D_SOD-123
- D39: renamed from D55; footprint Diodes_SMD:D_SOD-123 -> Diode_SMD:D_SOD-123
- D4: renamed from D18; footprint Diodes_SMD:D_SOD-123 -> Diode_SMD:D_SOD-123
- D41: renamed from D59; footprint Diodes_SMD:D_SOD-123 -> Diode_SMD:D_SOD-123
- D42: renamed from D60; footprint Diodes_SMD:D_SOD-123 -> Diode_SMD:D_SOD-123
- D43: renamed from D67; footprint Diodes_SMD:D_SOD-123 -> Diode_SMD:D_SOD-123
- D44: renamed from D58; footprint Diodes_SMD:D_SOD-123 -> Diode_SMD:D_SOD-123
- D45: renamed from D61; footprint Diodes_SMD:D_SOD-123 -> Diode_SMD:D_SOD-123
- D46: renamed from D62; footprint Diodes_SMD:D_SOD-123 -> Diode_SMD:D_SOD-123
- D47: renamed from D1; footprint Diodes_SMD:D_SOD-123 -> Diode_SMD:D_SOD-123
- D5: renamed from D19; footprint Diodes_SMD:D_SOD-123 -> Diode_SMD:D_SOD-123
- D6: renamed from D20; footprint Diodes_SMD:D_SOD-123 -> Diode_SMD:D_SOD-123
- D7: renamed from D21; footprint Diodes_SMD:D_SOD-123 -> Diode_SMD:D_SOD-123
- D8: renamed from D22; footprint Diodes_SMD:D_SOD-123 -> Diode_SMD:D_SOD-123
- D9: renamed from D23; footprint Diodes_SMD:D_SOD-123 -> Diode_SMD:D_SOD-123
- F1: footprint Fuse_Holders_and_Fuses:Fuse_SMD1206_Reflow -> Fuse:Fuse_1206_3216Metric
- K_,1, K_.1, K_;1, K_A1, K_B1, K_C1, K_D1, K_E1, K_F1, K_G1, K_H1, K_I1, K_J1, K_K1, K_L1, K_M1, K_N1, K_O1, K_P1, K_Q1, K_R1, K_S1, K_T1, K_U1, K_V1, K_W1, K_X1, K_Y1, K_Z1: footprint MX_Alps_Hybrid:MX-1U -> MX_Only:MXOnly-1U-Hotswap-Antishear; symbol MX_Alps_Hybrids:MX-1U -> MX_Alps_Hybrid:MX-NoLED
- K_ALT1: renamed from K_WIN1; footprint MX_Alps_Hybrid:MX-1U -> MX_Only:MXOnly-1U-Hotswap-Antishear; symbol MX_Alps_Hybrids:MX-1U -> MX_Alps_Hybrid:MX-NoLED
- K_ALT2: renamed from K_RALT1; footprint MX_Alps_Hybrid:MX-1.25U -> MX_Only:MXOnly-1U-Hotswap-Antishear; symbol MX_Alps_Hybrids:MX-1U -> MX_Alps_Hybrid:MX-NoLED
- K_CTRL1: footprint MX_Alps_Hybrid:MX-1.25U -> MX_Only:MXOnly-1U-Hotswap-Antishear; symbol MX_Alps_Hybrids:MX-1U -> MX_Alps_Hybrid:MX-NoLED
- K_ESC1: renamed from K_TAB1; footprint MX_Alps_Hybrid:MX-1.5U -> MX_Only:MXOnly-1U-Hotswap-Antishear; symbol MX_Alps_Hybrids:MX-1U -> MX_Alps_Hybrid:MX-NoLED
- K_SHIFT1: footprint MX_Alps_Hybrid:MX-2.25U -> MX_Only:MXOnly-1U-Hotswap-Antishear; symbol MX_Alps_Hybrids:MX-1U -> MX_Alps_Hybrid:MX-NoLED
- K_SHIFT2: renamed from K_RSHIFT1; footprint MX_Alps_Hybrid:MX-1.75U -> MX_Only:MXOnly-1U-Hotswap-Antishear; symbol MX_Alps_Hybrids:MX-1U -> MX_Alps_Hybrid:MX-NoLED
- K_SPC1: renamed from K_ALT1; footprint MX_Alps_Hybrid:MX-1.25U -> MX_Only:MXOnly-1U-Hotswap-Antishear; symbol MX_Alps_Hybrids:MX-1U -> MX_Alps_Hybrid:MX-NoLED
- K_SPC2: renamed from K_SPACE2; footprint MX_Alps_Hybrid:MX-6U-ReversedStabilizers -> MX_Only:MXOnly-1U-Hotswap-Antishear; symbol MX_Alps_Hybrids:MX-1U -> MX_Alps_Hybrid:MX-NoLED
- K_TAB1: renamed from K_CAPS1; footprint MX_Alps_Hybrid:MX-1.75U -> MX_Only:MXOnly-1U-Hotswap-Antishear; symbol MX_Alps_Hybrids:MX-1U -> MX_Alps_Hybrid:MX-NoLED
- K_WIN1: renamed from K_LSPACE1; footprint MX_Alps_Hybrid:MX-2.25U-ReversedStabilizers -> MX_Only:MXOnly-1U-Hotswap-Antishear; symbol MX_Alps_Hybrids:MX-1U -> MX_Alps_Hybrid:MX-NoLED
- K_WIN2: renamed from K_RSPACE1; footprint MX_Alps_Hybrid:MX-2.75U-ReversedStabilizers -> MX_Only:MXOnly-1U-Hotswap-Antishear; symbol MX_Alps_Hybrids:MX-1U -> MX_Alps_Hybrid:MX-NoLED
- R1: value 1k -> 100k
- R2: value 10k -> 100k
- SW1: renamed from SW2; footprint Buttons_Switches_SMD:SW_SPST_SKQG -> Button_Switch_SMD:SW_SPST_SKQG_WithoutStem
- U1: renamed from U4; footprint TO_SOT_Packages_SMD:SOT-23 -> Package_TO_SOT_SMD:SOT-23
- U2: renamed from U3; footprint Housings_DFN_QFN:QFN-48-1EP_7x7mm_Pitch0.5mm -> Package_QFP:LQFP-48_7x7mm_P0.5mm
- renumbered R73 to R3, R74 to R5
Connections:
- net labels added: BOOT0, COL12, COL13, NRST
- net labels removed: .-COL, .-LEDGND, .-ROW, LEDGND, RGBLED
- wire segments 534 -> 218
- no-connect marks 8 -> 11
Other:
- note added: "ESD_PROTECTION"
- note added: "MATRIX"
- note added: "MCU"
- note added: "POWER_SUPPLY"
- note added: "RESET"
- note added: "USB_PORT"
- moved on the sheet: C1, C10, C11, C2, C6, C7, C8, C9, D10, D11, D12, D13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
