File: Vision.kicad_pcb (KiCad board)
At the start: 2 copper layers, 244.5 x 76.2 mm, 193 parts, among them Q1 2N7002, SW2 SW_Push, SW3 SW_SPDT, U2 PRTR5V0U2X, U3 STM32F072CBUx, U4 MCP1700-3002E_SOT23

Commit message: Set switch position
Parts:
- removed C13, C14, C15, C16, C17, C18, C19, C20, C21, C22: 0.1uF, Capacitors_SMD:C_0603
- removed C23, C24: 4.7uF, Capacitors_SMD:C_0603
- removed C25, C26: 1uF, Capacitors_SMD:C_0603
- removed D52, D53, D54, D55, D58, D59, D60, D61, D62, D63, D64, D67: SOD-123, Diodes_SMD:D_SOD-123
- removed G***: LOGO, locallib:ai-4.8-ring
- removed G***: LOGO, locallib:ai-ring-6mm
- removed K_CAPS1, K_RSHIFT1, K_RSHIFT2: MX-1.75U, MX_Alps_Hybrid:MX-1.75U
- removed K_CAPS2: MX-1.25U, MX_Alps_Hybrid:MX-1.25U-FLIPPED
- removed K_ENTER2, K_RALT1, K_RCTRL1: MX-1.25U, MX_Alps_Hybrid:MX-1.25U
- removed K_ENTER3: MX-ISO, MX_Alps_Hybrid:MX-ISO-ReversedStabilizers
- removed K_LSPACE1: MX-2.25U, MX_Alps_Hybrid:MX-2.25U-ReversedStabilizers
- removed K_LSPACE2: MX-2.75U, MX_Alps_Hybrid:MX-2.75U-FLIPPED-ReversedStabilizers
- removed K_RSHIFT3, K_SHIFT3, K_SPACE3: MX-1U, MX_Alps_Hybrid:MX-1U
- removed K_RSHIFT4: MX-2.75U, MX_Alps_Hybrid:MX-2.75U
- removed K_RSPACE1: MX-2.75U, MX_Alps_Hybrid:MX-2.75U-ReversedStabilizers
- removed K_RSPACE2: MX-2.25U, MX_Alps_Hybrid:MX-2.25U-FLIPPED-ReversedStabilizers
- removed K_RWIN1: MX-1.25U, MX_Alps_Hybrid:MX-1U
- removed K_SPACE2: MX-6U, MX_Alps_Hybrid:MX-6U-ReversedStabilizers
- removed K_SPACE4: MX-1U, MX_Alps_Hybrid:MX-1U-FLIPPED
- removed K_\1: MX-1.5U, MX_Alps_Hybrid:MX-1.5U
- removed R16, R17, R18, R19, R20, R21, R22, R23, R24, R25, R26, R27, R31, R32, R33, R34, R35, R36, R37, R38, R39, R40, R41, R42, R44, R45, R46, R47, R48, R49, R50, R51, R52, R53, R54, R55, R58, R59, R60, R61, R62, R63, R64, R72: 1k, Resistors_SMD:R_0805
- removed R69: 100, Resistors_SMD:R_0805
- removed R73, R74: 5.1k, Resistors_SMD:R_0805
- removed RGB1, RGB10, RGB11, RGB12, RGB2, RGB3, RGB4, RGB5, RGB6, RGB7, RGB8, RGB9: WS2812B, LEDs:LED_WS2812B-PLCC4
- removed SW2: SW_Push, Buttons_Switches_SMD:SW_SPST_SKQG
- removed SW3: SW_SPDT, Buttons_Switches_SMD:SW_SPDT_PCM12
- removed U4: MCP1700-3002E_SOT23, TO_SOT_Packages_SMD:SOT-23
- added C2: 1uF, Capacitor_SMD:C_0603_1608Metric, F.Cu at (428.5, -254.7)
- added C3: 4.7nF, Capacitor_SMD:C_0603_1608Metric, F.Cu at (398.7, -222.2)
- added C4: 10uF, Capacitor_SMD:C_0603_1608Metric, F.Cu at (422.7, -253.9)
- added C6: 10nF, Capacitor_SMD:C_0603_1608Metric, F.Cu at (428.5, -257.2)
- added C7: 100nF, Capacitor_SMD:C_0603_1608Metric, F.Cu at (433.4, -259.5)
- added C8: 100nF, Capacitor_SMD:C_0603_1608Metric, F.Cu at (393.0, -218.9)
- added D10: SOD-123, Diode_SMD:D_SOD-123, F.Cu at (406.8, -236.6)
- added D11: SOD-123, Diode_SMD:D_SOD-123, F.Cu at (401.0, -226.6)
- added D12: SOD-123, Diode_SMD:D_SOD-123, F.Cu at (401.0, -229.9)
- added D13: SOD-123, Diode_SMD:D_SOD-123, F.Cu at (406.8, -233.3)
- added D14: SOD-123, Diode_SMD:D_SOD-123, F.Cu at (401.0, -233.3)
- added D15: SOD-123, Diode_SMD:D_SOD-123, F.Cu at (419.8, -246.7)
- added D2: SOD-123, Diode_SMD:D_SOD-123, F.Cu at (419.8, -250.1)
- added D28: SOD-123, Diode_SMD:D_SOD-123, F.Cu at (434.2, -277.0)
- added D29: SOD-123, Diode_SMD:D_SOD-123, F.Cu at (434.2, -267.0)
- added D3: SOD-123, Diode_SMD:D_SOD-123, F.Cu at (393.8, -221.8)
- added D30: SOD-123, Diode_SMD:D_SOD-123, F.Cu at (414.0, -240.0)
- added D4: SOD-123, Diode_SMD:D_SOD-123, F.Cu at (434.2, -273.7)
- added D43: SOD-123, Diode_SMD:D_SOD-123, F.Cu at (414.0, -243.4)
- added D5: SOD-123, Diode_SMD:D_SOD-123, F.Cu at (423.6, -256.8)
- added D6: SOD-123, Diode_SMD:D_SOD-123, F.Cu at (414.0, -246.7)
- added D7: SOD-123, Diode_SMD:D_SOD-123, F.Cu at (434.2, -270.3)
- added D8: SOD-123, Diode_SMD:D_SOD-123, F.Cu at (414.0, -250.1)
- added D9: SOD-123, Diode_SMD:D_SOD-123, F.Cu at (401.0, -236.6)
- added J1: Conn_ARM_JTAG_SWD_10, Connector_PinHeader_2.54mm:PinHeader_2x05_P2.54mm_Vertical, F.Cu at (393.3, -236.0)
- added K_ALT2: MX-1.5U, MX_Only:MXOnly-1.5U-Hotswap, F.Cu at (373.5, 2.40)
- added K_B2: MX-1U, MX_Only:MXOnly-1U-Hotswap, F.Cu at (312.7, -5.70)
- added K_BSPC1: MX-1U, MX_Only:MXOnly-1U-Hotswap, F.Cu at (404.5, -57.2)
- added K_CTRL2: MX-1.5U, MX_Only:MXOnly-1.5U-Hotswap, F.Cu at (423.6, -0.10)
- added K_DEL1: MX-1U, MX_Only:MXOnly-1U-Hotswap, F.Cu at (423.3, -57.2)
- added K_ESC1: MX-1U, MX_Only:MXOnly-1U-Hotswap, F.Cu at (178.0, -57.2)
- added K_FN1: MX-1U, MX_Only:MXOnly-1U-Hotswap, F.Cu at (432.0, -19.1)
- added K_PGDN1: MX-1U, MX_Only:MXOnly-1U-Hotswap, F.Cu at (150.9, -40.3)
- added K_PGUP1: MX-1U, MX_Only:MXOnly-1U-Hotswap, F.Cu at (154.9, -59.4)
- added K_SPC1: MX-2U, MX_Only:MXOnly-2U-Hotswap-ReversedStabilizers, F.Cu at (251.7, 7.87)
- added K_SPC2: MX-1.75U, MX_Only:MXOnly-1.75U-Hotswap, F.Cu at (323.7, 11.4)
- added K_WIN2: MX-1U, MX_Only:MXOnly-1U-Hotswap, F.Cu at (349.3, 6.00)
- added R4: 1M, Resistor_SMD:R_0603_1608Metric, F.Cu at (346.9, -247.9)
- added R5: 5.1k, Resistor_SMD:R_0603_1608Metric, F.Cu at (346.9, -245.4)
- added R6: 100k, Resistor_SMD:R_0603_1608Metric, F.Cu at (350.9, -247.9)
- added SW1: SW_Push, Button_Switch_SMD:SW_SPST_SKQG_WithoutStem, F.Cu at (415.9, -255.1)
- added U1: MCP1700-3002E_SOT23, Package_TO_SOT_SMD:SOT-23, F.Cu at (433.6, -263.0)
- C1, C10: value 0.1uF -> 1uF; footprint Capacitors_SMD:C_0603 -> Capacitor_SMD:C_0603_1608Metric
- C11, C12, C5: value 0.1uF -> 4.7uF; footprint Capacitors_SMD:C_0603 -> Capacitor_SMD:C_0603_1608Metric
- C9: value 0.1uF -> 100nF; footprint Capacitors_SMD:C_0603 -> Capacitor_SMD:C_0603_1608Metric
- D1, D16, D17, D18, D19, D20, D21, D22, D23, D24, D25, D26, D27, D31, D32, D33, D34, D35, D36, D37, D38, D39, D40, D41, D42, D44, D45, D46, D47, D48: footprint Diodes_SMD:D_SOD-123 -> Diode_SMD:D_SOD-123
- D49: value SOD-123 -> BAT41ZFILM; footprint Diodes_SMD:D_SOD-123 -> Diode_SMD:D_SOD-123
- D50: value SOD-123 -> SMF9.0CA; footprint Diodes_SMD:D_SOD-123 -> Diode_SMD:D_SOD-123
- D51: value SOD-123 -> 1N4148W; footprint Diodes_SMD:D_SOD-123 -> Diode_SMD:D_SOD-123
- F1: footprint Fuse_Holders_and_Fuses:Fuse_SMD1206_Reflow -> Fuse:Fuse_1206_3216Metric
- K_,1, K_.1, K_;1, K_A1, K_B1, K_C1, K_D1, K_E1, K_F1, K_G1, K_H1, K_I1, K_J1, K_K1, K_L1, K_M1, K_N1, K_O1, K_P1, K_Q1, K_R1, K_S1, K_T1, K_U1, K_V1, K_W1, K_WIN1, K_X1, K_Y1, K_Z1: footprint MX_Alps_Hybrid:MX-1U -> MX_Only:MXOnly-1U-Hotswap
- K_ALT1, K_CTRL1: value MX-1.25U -> MX-1.5U; footprint MX_Alps_Hybrid:MX-1.25U -> MX_Only:MXOnly-1.5U-Hotswap
- K_ENTER1, K_SHIFT1: value MX-2.25U -> MX-1.75U; footprint MX_Alps_Hybrid:MX-2.25U -> MX_Only:MXOnly-1.75U-Hotswap
- K_SHIFT2: footprint MX_Alps_Hybrid:MX-1.25U -> MX_Only:MXOnly-1.25U-Hotswap
- K_TAB1: value MX-1.5U -> MX-1.25U; footprint MX_Alps_Hybrid:MX-1.5U -> MX_Only:MXOnly-1.25U-Hotswap
- Q1: value 2N7002 -> DTC123J; footprint TO_SOT_Packages_SMD:SOT-23 -> Package_TO_SOT_SMD:SC-59
- R1: value 1k -> 100k; footprint Resistors_SMD:R_0805 -> Resistor_SMD:R_0603_1608Metric
- R2: value 10k -> 100k; footprint Resistors_SMD:R_0805 -> Resistor_SMD:R_0603_1608Metric
- R3: footprint Resistors_SMD:R_0805 -> Resistor_SMD:R_0603_1608Metric
- U2: value PRTR5V0U2X -> STM32F072CBUx; footprint random-keyboard-parts:SOT143B -> Package_QFP:LQFP-48_7x7mm_P0.5mm
- U3: value STM32F072CBUx -> TPD4E05U06DQAR; footprint Housings_DFN_QFN:QFN-48-1EP_7x7mm_Pitch0.5mm -> random-keyboard-parts:USON-TPDxE05U06
- moved K_SHIFT2 378.0 mm to (410.6, -19.1)
- moved C1 264.3 mm to (47.3, -215.0)
- moved C10 264.3 mm to (179.9, -215.0)
- moved C11 264.3 mm to (218.0, -215.0)
- moved C12 264.3 mm to (264.0, -219.0)
- moved C5 264.3 mm to (100.5, -215.0)
- moved C9 264.3 mm to (133.8, -215.0)
- moved D1 264.3 mm to (239.4, -169.0)
- moved D16 264.3 mm to (44.9, -226.1)
- moved D17 264.3 mm to (84.6, -226.1)
- moved D18 264.3 mm to (103.7, -226.1)
- moved D19 264.3 mm to (122.7, -226.1)
- moved D20 264.3 mm to (141.8, -226.1)
- moved D21 264.3 mm to (160.8, -226.1)
- moved D22 264.3 mm to (179.9, -226.1)
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Connections:
- C1 pad 1: GND -> +5V
- C1 pad 2: +5V -> GND
- C10 pad 1: GND -> +3V3
- C10 pad 2: +5V -> GND
- C11 pad 1: GND -> +3V3
- C11 pad 2: +5V -> GND
- C12 pad 1: GND -> +3V3
- C12 pad 2: +5V -> GND
- C5 pad 1: GND -> NRST
- C5 pad 2: +5V -> GND
- C9 pad 1: GND -> +3V3
- C9 pad 2: +5V -> GND
- D1 pad 1: ROW3 -> ROW0
- D16 pad 1: ROW0 -> ROW1
- D17 pad 1: ROW0 -> ROW1
- D18 pad 1: ROW0 -> ROW1
- D19 pad 1: ROW0 -> ROW1
- D20 pad 1: ROW0 -> ROW1
- D21 pad 1: ROW0 -> ROW1
- D22 pad 1: ROW0 -> ROW1
- D23 pad 1: ROW0 -> ROW1
- D24 pad 1: ROW0 -> ROW1
- D25 pad 1: ROW0 -> ROW1
- D26 pad 1: ROW0 -> ROW1
- D27 pad 1: ROW0 -> ROW1
- D31 pad 1: ROW1 -> ROW2
- D32 pad 1: ROW1 -> ROW2
- D33 pad 1: ROW1 -> ROW2
- D34 pad 1: ROW1 -> ROW2
- D35 pad 1: ROW1 -> ROW2
- D36 pad 1: ROW1 -> ROW2
- D37 pad 1: ROW1 -> ROW2
- D38 pad 1: ROW1 -> ROW2
- D39 pad 1: ROW1 -> ROW2
- D40 pad 1: ROW1 -> ROW2
- D41 pad 1: ROW1 -> ROW3
- D42 pad 1: ROW1 -> ROW3
- D44 pad 1: ROW2 -> ROW3
- D45 pad 1: ROW2 -> ROW3
- D46 pad 1: ROW2 -> ROW3
- D47 pad 1: ROW2 -> ROW3
- D48 pad 1: ROW2 -> ROW3
- D49 pad 1: ROW2 -> +5V
- D49 pad 2: Net-(D49-Pad2) -> +3V3
- D50 pad 1: ROW2 -> +5V
- D50 pad 2: Net-(D50-Pad2) -> GND
- D51 pad 1: ROW2 -> BOOT0
- K_,1 pad 1: COL9 -> COL10
- K_,1 pad 2: Net-(D53-Pad2) -> Net-(D37-Pad2)
- K_.1 pad 1: .-COL -> COL11
- K_.1 pad 2: .-ROW -> Net-(D38-Pad2)
- K_;1 pad 1: .-COL -> COL11
- K_;1 pad 2: Net-(D41-Pad2) -> Net-(D26-Pad2)
- K_A1 pad 1: COL1 -> COL2
- K_A1 pad 2: Net-(D32-Pad2) -> Net-(D17-Pad2)
- K_ALT1 pad 1: COL2 -> COL3
- K_ALT1 pad 2: Net-(D67-Pad2) -> Net-(D42-Pad2)
- K_B1 pad 2: Net-(D50-Pad2) -> Net-(D33-Pad2)
- K_C1 pad 2: Net-(D48-Pad2) -> Net-(D31-Pad2)
- K_CTRL1 pad 1: COL0 -> COL1
- K_CTRL1 pad 2: Net-(D59-Pad2) -> Net-(D41-Pad2)
- K_D1 pad 1: COL3 -> COL4
- K_D1 pad 2: Net-(D34-Pad2) -> Net-(D19-Pad2)
- K_E1 pad 1: COL3 -> COL4
- K_E1 pad 2: Net-(D19-Pad2) -> Net-(D5-Pad2)
- K_ENTER1 pad 1: COL11 -> COL13
- K_ENTER1 pad 2: Net-(D42-Pad2) -> Net-(D27-Pad2)
- K_F1 pad 1: COL4 -> COL5
- K_F1 pad 2: Net-(D35-Pad2) -> Net-(D20-Pad2)
- K_G1 pad 1: COL5 -> COL6
- K_G1 pad 2: Net-(D36-Pad2) -> Net-(D21-Pad2)
- K_H1 pad 1: COL6 -> COL7
- K_H1 pad 2: Net-(D37-Pad2) -> Net-(D22-Pad2)
- K_I1 pad 1: COL8 -> COL9
- K_I1 pad 2: Net-(D24-Pad2) -> Net-(D10-Pad2)
- K_J1 pad 1: COL7 -> COL8
- K_J1 pad 2: Net-(D38-Pad2) -> Net-(D23-Pad2)
- K_K1 pad 1: COL8 -> COL9
- K_K1 pad 2: Net-(D39-Pad2) -> Net-(D24-Pad2)
- K_L1 pad 1: COL9 -> COL10
- K_L1 pad 2: Net-(D40-Pad2) -> Net-(D25-Pad2)
- K_M1 pad 1: COL8 -> COL9
- K_M1 pad 2: Net-(D52-Pad2) -> Net-(D36-Pad2)
- K_N1 pad 1: COL7 -> COL8
- K_N1 pad 2: Net-(D51-Pad2) -> Net-(D35-Pad2)
- K_O1 pad 1: COL9 -> COL10
- K_O1 pad 2: Net-(D25-Pad2) -> Net-(D11-Pad2)
- K_P1 pad 1: .-COL -> COL11
- K_P1 pad 2: Net-(D26-Pad2) -> Net-(D12-Pad2)
- K_Q1 pad 1: COL1 -> COL2
- K_Q1 pad 2: Net-(D17-Pad2) -> Net-(D3-Pad2)
- K_R1 pad 1: COL4 -> COL5
- K_R1 pad 2: Net-(D20-Pad2) -> Net-(D6-Pad2)
- K_S1 pad 1: COL2 -> COL3
- K_S1 pad 2: Net-(D33-Pad2) -> Net-(D18-Pad2)
- K_SHIFT1 pad 1: COL0 -> COL1
- K_SHIFT1 pad 2: Net-(D45-Pad2) -> Net-(D28-Pad2)
- K_SHIFT2 pad 1: COL0 -> COL12
- K_SHIFT2 pad 2: Net-(D45-Pad2) -> Net-(D39-Pad2)
- K_T1 pad 1: COL5 -> COL6
- K_T1 pad 2: Net-(D21-Pad2) -> Net-(D7-Pad2)
- K_TAB1 pad 1: COL0 -> COL1
- K_U1 pad 1: COL7 -> COL8
- K_U1 pad 2: Net-(D23-Pad2) -> Net-(D9-Pad2)
- K_V1 pad 2: Net-(D49-Pad2) -> Net-(D32-Pad2)
- K_W1 pad 1: COL2 -> COL3
- K_W1 pad 2: Net-(D18-Pad2) -> Net-(D4-Pad2)
- K_WIN1 pad 1: COL1 -> COL6
- K_WIN1 pad 2: Net-(D60-Pad2) -> Net-(D44-Pad2)
- K_X1 pad 2: Net-(D47-Pad2) -> Net-(D30-Pad2)
- K_Y1 pad 1: COL6 -> COL7
- K_Y1 pad 2: Net-(D22-Pad2) -> Net-(D8-Pad2)
- K_Z1 pad 2: Net-(D46-Pad2) -> Net-(D29-Pad2)
- Q1 pad 1: Net-(Q1-Pad1) -> Net-(D51-Pad2)
- Q1 pad 3: LEDGND -> NRST
- R1 pad 1: Net-(K_RALT1-Pad4) -> GND
- R1 pad 2: LEDGND -> +5V
- R2 pad 1: Net-(R2-Pad1) -> GND
- R2 pad 2: Net-(R2-Pad2) -> +3V3
- R3 pad 2: Net-(Q1-Pad1) -> Net-(R3-Pad2)
- U2 pad 1: GND -> +3V3
- U2 pad 2: D+ -> (no net)
- U2 pad 3: D- -> (no net)
- U2 pad 4: VCC -> (no net)
- U3 pad 1: +3V3 -> D+
- U3 pad 10: COL11 -> D+
- U3 pad 2: Net-(U3-Pad2) -> D-
- U3 pad 3: Net-(U3-Pad3) -> GND
- U3 pad 4: Net-(U3-Pad4) -> D+
- U3 pad 5: Net-(U3-Pad5) -> D-
- U3 pad 6: Net-(U3-Pad6) -> D-
- U3 pad 7: Net-(SW2-Pad2) -> D+
- U3 pad 9: +3V3 -> D-
- USB1 pad 13: GND -> Net-(C3-Pad2)
- USB1 pad 3: Net-(USB1-Pad3) -> (no net)
- USB1 pad 4: Net-(R73-Pad2) -> Net-(R3-Pad2)
- USB1 pad 9: Net-(USB1-Pad9) -> (no net)
Routing:
- net +5V: track 1239.1 -> 0.00 mm, vias 17 -> 0
- net LEDGND: track 850.8 -> 0.00 mm, vias 9 -> 0
- net GND: track 704.9 -> 0.00 mm, vias 17 -> 0
- net COL11: track 320.7 -> 0.00 mm
- net ROW3: track 288.0 -> 0.00 mm, vias 4 -> 0
- net .-COL: track 261.5 -> 0.00 mm, vias 2 -> 0
- net ROW0: track 246.6 -> 0.00 mm, vias 3 -> 0
- net ROW1: track 226.2 -> 0.00 mm, vias 3 -> 0
- net COL9: track 221.4 -> 0.00 mm
- net ROW2: track 221.3 -> 0.00 mm, vias 4 -> 0
- net COL8: track 213.0 -> 0.00 mm
- net COL6: track 187.4 -> 0.00 mm
- net COL7: track 162.8 -> 0.00 mm
- net COL4: track 138.1 -> 0.00 mm
- net COL5: track 128.3 -> 0.00 mm
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Other:
- board outline removed
- board text added: "VISION"
- board text removed: "40"
- board text removed: "VOYAGER"
- board text removed: "Voyager40 PCB Rev 2.0 20190217"
- board text removed: "kb.ai03.me"
