File: Vision.kicad_pcb (KiCad board)
At the start: 2 copper layers, 125 parts, among them J1 Conn_ARM_JTAG_SWD_10, Q1 DTC123J, SW1 SW_Push, U1 MCP1700-3002E_SOT23, U2 STM32F072CBUx, U3 TPD4E05U06DQAR

Commit message: Fix switch position
Parts:
- D10, D11, D12, D13, D14, D15, D2, D28, D29, D3, D30, D4, D43, D5, D6, D7, D8, D9: moved to B.Cu
- moved D28 535.5 mm to (100.4, 141.7), turned to 90 degrees
- moved D29 511.5 mm to (126.6, 141.7), turned to 90 degrees
- moved D15 504.1 mm to (74.4, 120.5), turned to 90 degrees
- moved D4 479.0 mm to (140.6, 104.8), turned to 78 degrees
- moved D43 478.0 mm to (175.1, 170.6), turned to 78 degrees
- moved D2 475.8 mm to (101.5, 103.6), turned to 90 degrees
- moved D30 468.8 mm to (146.6, 145.0), turned to 78 degrees
- moved D7 454.2 mm to (196.5, 116.7), turned to 78 degrees
- moved D5 451.1 mm to (159.2, 108.8), turned to 78 degrees
- moved J1 433.2 mm to (211.8, 157.4)
- moved D6 430.1 mm to (177.8, 112.7), turned to 78 degrees
- moved D3 425.0 mm to (120.6, 103.6), turned to 90 degrees
- moved D8 407.5 mm to (233.2, 115.1), turned to 102 degrees
- moved D48 407.2 mm to (347.1, 160.8)
- moved D41 396.1 mm to (98.0, 160.8)
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Routing:
- removed copper zone on B.Cu, net GND
Other:
- board outline added: 300.1 x 99.9 mm

Commit message: Route PCB
Parts:
- added C13: 100nF, Capacitor_SMD:C_0603_1608Metric, B.Cu at (213.6, 137.6)
- added H1: LOGO1, locallib:logo1, B.Cu at (68.8, 141.5)
- added H2: LOGO2, locallib:logo2, F.Cu at (68.5, 148.4)
- C2, C3, C4, C6, C7, C8, J1, R4, R5, R6, SW1, U1: moved to B.Cu
- moved C10 126.1 mm to (209.0, 139.5), turned to 0 degrees
- moved Q1 114.8 mm to (208.3, 147.8), turned to 90 degrees
- moved C8 110.9 mm to (214.4, 125.6), turned to 90 degrees
- moved C5 108.6 mm to (208.3, 144.4), turned to 180 degrees
- moved D51 105.1 mm to (212.8, 147.9), turned to 270 degrees
- moved SW1 99.7 mm to (209.9, 155.4), turned to 270 degrees
- moved C9 99.2 mm to (216.2, 134.6), turned to 90 degrees
- moved C3 97.3 mm to (218.6, 89.0), turned to 90 degrees
- moved C11 93.0 mm to (201.8, 128.3)
- moved C1 89.9 mm to (206.3, 101.3), turned to 0 degrees
- moved C12 87.7 mm to (216.2, 125.6), turned to 90 degrees
- moved C4 87.4 mm to (213.6, 144.4), turned to 180 degrees
- moved C6 84.8 mm to (209.0, 137.8)
- moved R1 83.6 mm to (206.3, 99.3), turned to 180 degrees
- moved D50 82.6 mm to (202.8, 94.8)
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Connections:
- U2 pad 10: COL11 -> (no net)
- U2 pad 11: COL10 -> ROW3
- U2 pad 12: COL9 -> ROW2
- U2 pad 13: COL8 -> COL6
- U2 pad 14: COL7 -> COL5
- U2 pad 15: COL6 -> COL4
- U2 pad 16: (no net) -> COL3
- U2 pad 17: COL5 -> COL2
- U2 pad 18: COL4 -> COL1
- U2 pad 19: COL3 -> COL0
- U2 pad 20: COL2 -> ROW1
- U2 pad 21: COL1 -> (no net)
- U2 pad 22: ROW1 -> (no net)
- U2 pad 25: (no net) -> ROW0
- U2 pad 29: ROW2 -> (no net)
- U2 pad 30: ROW3 -> (no net)
- U2 pad 31: COL0 -> (no net)
- U2 pad 38: ROW0 -> COL13
- U2 pad 40: COL13 -> COL11
- U2 pad 41: (no net) -> COL10
- U2 pad 42: (no net) -> COL9
- U2 pad 43: (no net) -> COL8
- U2 pad 45: (no net) -> COL7
Routing:
- net ROW3: track 0.00 -> 299.6 mm, vias 0 -> 2
- net ROW0: track 0.00 -> 295.3 mm, vias 0 -> 2
- net ROW1: track 0.00 -> 292.0 mm, vias 0 -> 2
- net ROW2: track 0.00 -> 277.2 mm
- net COL13: track 0.00 -> 206.5 mm, vias 0 -> 4
- net COL1: track 0.00 -> 195.5 mm, vias 0 -> 3
- net COL0: track 0.00 -> 182.1 mm
- net GND: track 0.00 -> 175.5 mm, vias 0 -> 6
- net COL3: track 0.00 -> 156.0 mm, vias 0 -> 4
- net COL12: track 0.00 -> 155.2 mm, vias 0 -> 2
- net +3V3: track 0.00 -> 151.6 mm, vias 0 -> 7
- net COL2: track 0.00 -> 150.5 mm, vias 0 -> 3
- net COL10: track 0.00 -> 143.3 mm, vias 0 -> 4
- net COL11: track 0.00 -> 140.5 mm, vias 0 -> 3
- net COL9: track 0.00 -> 119.0 mm, vias 0 -> 4
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- added copper zone on B.Cu, net GND
- added copper zone on B.Cu, net Net-(C3-Pad2)
Other:
- board text added: "3V3"
- board text added: "GND"
- board text added: "NRST"
- board text added: "PCBv1.0 by SatT"
- board text added: "SWCLK"
- board text added: "SWDIO"

Commit message: Add edgerails
Parts:
- added H10: MOUSEBITES, random-keyboard-parts:breakaway-mousebites, F.Cu at (259.0, 85.5)
- added H11: MOUSEBITES, random-keyboard-parts:breakaway-mousebites, F.Cu at (161.0, 85.5)
- added H12: MOUSEBITES, random-keyboard-parts:breakaway-mousebites, F.Cu at (68.3, 85.5)
- added H13: MOUSEBITES, random-keyboard-parts:breakaway-mousebites, F.Cu at (78.3, 164.0)
- added H14: MOUSEBITES, random-keyboard-parts:breakaway-mousebites, F.Cu at (149.5, 170.4)
- added H15: MOUSEBITES, random-keyboard-parts:breakaway-mousebites, F.Cu at (210.0, 181.3)
- added H3: FIDUCIAL, Fiducial:Fiducial_0.75mm_Mask2.25mm, F.Cu at (340.4, 73.0)
- added H4: FIDUCIAL, Fiducial:Fiducial_0.75mm_Mask2.25mm, F.Cu at (75.3, 189.3)
- added H5: FIDUCIAL, Fiducial:Fiducial_1mm_Mask3mm, F.Cu at (75.3, 73.0)
- added H6: FIDUCIAL, Fiducial:Fiducial_1mm_Mask3mm, F.Cu at (340.4, 189.3)
- added H7: MOUSEBITES, random-keyboard-parts:breakaway-mousebites, F.Cu at (276.1, 169.1)
- added H8: MOUSEBITES, random-keyboard-parts:breakaway-mousebites, F.Cu at (332.4, 164.0)
- added H9: MOUSEBITES, random-keyboard-parts:breakaway-mousebites, F.Cu at (342.4, 85.5)
Other:
- board size 300.1 x 99.9 mm -> 300.1 x 126.3 mm
