File: Vision.kicad_pcb (KiCad board)
At the start: 2 copper layers, 300.1 x 126.3 mm, 141 parts, among them J1 Conn_ARM_JTAG_SWD_10, Q1 DTC123J, SW1 SW_Push, U1 MCP1700-3002E_SOT23, U2 STM32F072CBUx, U3 TPD4E05U06DQAR

Commit message: Fix fiducials
Parts:
- H3, H4, H5, H6: moved to B.Cu
Changed lines of the file:
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@@
     (pad "" np_thru_hole circle (at 0 -0.254 12) (size 0.7874 0.7874) (drill 0.7874) (layers *.Cu *.Mask))
   )
-  (module Fiducial:Fiducial_1mm_Mask3mm (layer F.Cu)
+  (module Fiducial:Fiducial_1mm_Mask3mm (layer B.Cu)
     (at 340.407501 189.34088)
     (descr "Circular Fiducial, 1mm bare copper, 3mm soldermask opening (recommended)")
     (tags fiducial)
     (attr smd)
-    (fp_text reference H6 (at 0 -2.54) (layer F.SilkS)
-      (effects (font (size 1 1) (thickness 0.15)))
+    (fp_text reference H6 (at 0 2.54) (layer B.SilkS) hide
+      (effects (font (size 1 1) (thickness 0.15)) (justify mirror))
     )
-    (fp_text value FIDUCIAL (at 0 2.286) (layer F.Fab)
-      (effects (font (size 1 1) (thickness 0.15)))
+    (fp_text value FIDUCIAL (at 0 -2.286) (layer B.Fab)
+      (effects (font (size 1 1) (thickness 0.15)) (justify mirror))
     )
-    (fp_circle (center 0 0) (end 1.75 0) (layer F.CrtYd) (width 0.05))
-    (fp_text user %R (at 0 0) (layer F.Fab)
-      (effects (font (size 0.4 0.4) (thickness 0.06)))
+    (fp_circle (center 0 0) (end 1.75 0) (layer B.CrtYd) (width 0.05))
+    (fp_text user %R (at 0 0) (layer B.Fab)
+      (effects (font (size 0.4 0.4) (thickness 0.06)) (justify mirror))
     )
-    (fp_circle (center 0 0) (end 1.5 0) (layer F.Fab) (width 0.1))
-    (pad "" smd circle (at 0 0) (size 1 1) (layers F.Cu F.Mask)
+    (fp_circle (center 0 0) (end 1.5 0) (layer B.Fab) (width 0.1))
+    (pad "" smd circle (at 0 0) (size 1 1) (layers B.Cu B.Mask)
       (solder_mask_margin 1) (clearance 1))
   )
-  (module Fiducial:Fiducial_1mm_Mask3mm (layer F.Cu)
+  (module Fiducial:Fiducial_1mm_Mask3mm (layer B.Cu)
     (at 75.265001 73)
     (descr "Circular Fiducial, 1mm bare copper, 3mm soldermask opening (recommended)")
     (tags fiducial)
     (attr smd)
-    (fp_text reference H5 (at 0 -2.54) (layer F.SilkS)
-      (effects (font (size 1 1) (thickness 0.15)))
+    (fp_text reference H5 (at 0 2.54) (layer B.SilkS) hide
+      (effects (font (size 1 1) (thickness 0.15)) (justify mirror))
     )
-    (fp_text value FIDUCIAL (at 0 2.286) (layer F.Fab)
-      (effects (font (size 1 1) (thickness 0.15)))
+    (fp_text value FIDUCIAL (at 0 -2.286) (layer B.Fab)
+      (effects (font (size 1 1) (thickness 0.15)) (justify mirror))
     )
-    (fp_circle (center 0 0) (end 1.75 0) (layer F.CrtYd) (width 0.05))
-    (fp_text user %R (at 0 0) (layer F.Fab)
-      (effects (font (size 0.4 0.4) (thickness 0.06)))
+    (fp_circle (center 0 0) (end 1.75 0) (layer B.CrtYd) (width 0.05))
+    (fp_text user %R (at 0 0) (layer B.Fab)
+      (effects (font (size 0.4 0.4) (thickness 0.06)) (justify mirror))
     )
-    (fp_circle (center 0 0) (end 1.5 0) (layer F.Fab) (width 0.1))
-    (pad "" smd circle (at 0 0) (size 1 1) (layers F.Cu F.Mask)
+    (fp_circle (center 0 0) (end 1.5 0) (layer B.Fab) (width 0.1))
+    (pad "" smd circle (at 0 0) (size 1 1) (layers B.Cu B.Mask)
       (solder_mask_margin 1) (clearance 1))
   )
-  (module Fiducial:Fiducial_0.75mm_Mask2.25mm (layer F.Cu)
+  (module Fiducial:Fiducial_0.75mm_Mask2.25mm (layer B.Cu)
     (at 75.265002 189.34088)
     (descr "Circular Fiducial, 0.75mm bare copper, 2.25mm soldermask opening")
     (tags fiducial)
     (attr smd)
-    (fp_text reference H4 (at 0 -2.0955) (layer F.SilkS)
-      (effects (font (size 1 1) (thickness 0.15)))
+    (fp_text reference H4 (at 0 2.0955) (layer B.SilkS) hide
+      (effects (font (size 1 1) (thickness 0.15)) (justify mirror))
     )
-    (fp_text value FIDUCIAL (at 0 2.032) (layer F.Fab)
-      (effects (font (size 1 1) (thickness 0.15)))
+    (fp_text value FIDUCIAL (at 0 -2.032) (layer B.Fab)
+      (effects (font (size 1 1) (thickness 0.15)) (justify mirror))
     )
-    (fp_circle (center 0 0) (end 1.38 0) (layer F.CrtYd) (width 0.05))
-    (fp_text user %R (at 0 0) (layer F.Fab)
-      (effects (font (size 0.3 0.3) (thickness 0.05)))
+    (fp_circle (center 0 0) (end 1.38 0) (layer B.CrtYd) (width 0.05))
+    (fp_text user %R (at 0 0) (layer B.Fab)
+      (effects (font (size 0.3 0.3) (thickness 0.05)) (justify mirror))
     )
-    (fp_circle (center 0 0) (end 1.125 0) (layer F.Fab) (width 0.1))
-    (pad "" smd circle (at 0 0) (size 0.75 0.75) (layers F.Cu F.Mask)
+    (fp_circle (center 0 0) (end 1.125 0) (layer B.Fab) (width 0.1))
+    (pad "" smd circle (at 0 0) (size 0.75 0.75) (layers B.Cu B.Mask)
       (solder_mask_margin 0.75) (clearance 0.75))
   )
-  (module Fiducial:Fiducial_0.75mm_Mask2.25mm (layer F.Cu)
+  (module Fiducial:Fiducial_0.75mm_Mask2.25mm (layer B.Cu)
     (at 340.4075 73)
     (descr "Circular Fiducial, 0.75mm bare copper, 2.25mm soldermask opening")
     (tags fiducial)
     (attr smd)
-    (fp_text reference H3 (at 0 -2.0955) (layer F.SilkS)
-      (effects (font (size 1 1) (thickness 0.15)))
+    (fp_text reference H3 (at 0 2.0955) (layer B.SilkS) hide
+      (effects (font (size 1 1) (thickness 0.15)) (justify mirror))
     )
-    (fp_text value FIDUCIAL (at 0 2.032) (layer F.Fab)
-      (effects (font (size 1 1) (thickness 0.15)))
+    (fp_text value FIDUCIAL (at 0 -2.032) (layer B.Fab)
+      (effects (font (size 1 1) (thickness 0.15)) (justify mirror))
     )
-    (fp_circle (center 0 0) (end 1.38 0) (layer F.CrtYd) (width 0.05))
-    (fp_text user %R (at 0 0) (layer F.Fab)
-      (effects (font (size 0.3 0.3) (thickness 0.05)))
+    (fp_circle (center 0 0) (end 1.38 0) (layer B.CrtYd) (width 0.05))
+    (fp_text user %R (at 0 0) (layer B.Fab)
+      (effects (font (size 0.3 0.3) (thickness 0.05)) (justify mirror))
     )
-    (fp_circle (center 0 0) (end 1.125 0) (layer F.Fab) (width 0.1))
-    (pad "" smd circle (at 0 0) (size 0.75 0.75) (layers F.Cu F.Mask)
+    (fp_circle (center 0 0) (end 1.125 0) (layer B.Fab) (width 0.1))
+    (pad "" smd circle (at 0 0) (size 0.75 0.75) (layers B.Cu B.Mask)
       (solder_mask_margin 0.75) (clearance 0.75))
   )

Commit message: Add BOM
Parts:
- D1, D10, D11, D12, D13, D14, D15, D16, D17, D18, D19, D2, D20, D21, D22, D23, D24, D25, D26, D27, D28, D29, D3, D30, D31, D32, D33, D34, D35, D36, D37, D38, D39, D4, D40, D41, D42, D43, D44, D45, D46, D47, D48, D5, D6, D7, D8, D9: value SOD-123 -> 1N4148W
- Q1: footprint Package_TO_SOT_SMD:SC-59 -> Package_TO_SOT_SMD:SOT-23

Commit message: Update pcb shape
Parts:
- moved H15 4.00 mm to (210.0, 177.3)
- moved H6 2.34 mm to (340.0, 187.0)
- moved H4 2.34 mm to (75.7, 187.0)
- moved H8 0.45 mm to (332.0, 164.0)
- moved H12 0.45 mm to (68.7, 85.5)
- moved H13 0.45 mm to (78.7, 164.0)
- moved H5 0.45 mm to (75.7, 73.0)
- moved H3 0.45 mm to (340.0, 73.0)
- moved H9 0.45 mm to (342.0, 85.5)
- moved H14 0.28 mm to (149.8, 170.4)
- moved H7 0.25 mm to (275.9, 169.1)
Other:
- board size 300.1 x 126.3 mm -> 299.2 x 124 mm

Commit message: Update revision number
Other:
- board text added: "PCBv1.1 by SatT"
- board text removed: "PCBv1.0 by SatT"
Changed lines of the file:
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@@
     (add_net "Net-(D8-Pad2)")
     (add_net "Net-(D9-Pad2)")
-    (add_net "Net-(J1-Pad6)")
-    (add_net "Net-(J1-Pad7)")
-    (add_net "Net-(J1-Pad8)")
     (add_net "Net-(R3-Pad2)")
     (add_net "Net-(R5-Pad2)")
-    (add_net "Net-(U2-Pad10)")
-    (add_net "Net-(U2-Pad2)")
-    (add_net "Net-(U2-Pad21)")
-    (add_net "Net-(U2-Pad22)")
-    (add_net "Net-(U2-Pad26)")
-    (add_net "Net-(U2-Pad27)")
-    (add_net "Net-(U2-Pad28)")
-    (add_net "Net-(U2-Pad29)")
-    (add_net "Net-(U2-Pad3)")
-    (add_net "Net-(U2-Pad30)")
-    (add_net "Net-(U2-Pad31)")
-    (add_net "Net-(U2-Pad4)")
-    (add_net "Net-(U2-Pad46)")
-    (add_net "Net-(U2-Pad5)")
-    (add_net "Net-(U2-Pad6)")
-    (add_net "Net-(USB1-Pad3)")
-    (add_net "Net-(USB1-Pad9)")
     (add_net ROW0)
     (add_net ROW1)
@@
     (effects (font (size 2.5 2.5) (thickness 0.2)) (justify left))
   )
-  (gr_text "PCBv1.0 by SatT" (at 70.3 143.7 90) (layer F.Cu)
+  (gr_text "PCBv1.1 by SatT" (at 70.3 143.7 90) (layer F.Cu)
     (effects (font (size 1 1) (thickness 0.15)) (justify left))
   )
-  (gr_text "PCBv1.0 by SatT" (at 70.3 143.7 90) (layer F.Mask)
+  (gr_text "PCBv1.1 by SatT" (at 70.3 143.7 90) (layer F.Mask)
     (effects (font (size 1 1) (thickness 0.15)) (justify left))
   )

Commit message: Fix routing
Routing:
- net ROW3: track 299.6 -> 303.7 mm
Changed lines of the file:
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@@
     (mod_text_size 1 1)
     (mod_text_width 0.15)
-    (pad_size 0.3 1.475)
-    (pad_drill 0)
+    (pad_size 5 5)
+    (pad_drill 3.048)
     (pad_to_mask_clearance 0.2)
     (aux_axis_origin 0 0)
@@
       (drillshape 0)
       (scaleselection 1)
-      (outputdirectory "./"))
+      (outputdirectory "Gerbers/"))
   )
   (net 0 "")
@@
   (gr_circle (center 214.25 135.6) (end 214.55 135.6) (layer B.SilkS) (width 0.15))
   (gr_circle (center 214.25 135.6) (end 214.55 135.6) (layer B.Fab) (width 0.15))
-  (gr_circle (center 210 170.84088) (end 208.9 170.84088) (layer Edge.Cuts) (width 0.2))
+  (gr_circle (center 210 170.84088) (end 211.1 170.84088) (layer Edge.Cuts) (width 0.2))
   (gr_circle (center 110.884935 157.540592) (end 109.784935 157.540592) (layer Edge.Cuts) (width 0.2))
   (gr_arc (start 297.613758 86.45) (end 298.085348 85.568181) (angle -28.13752657) (layer Edge.Cuts) (width 0.2))
@@
   (gr_circle (center 351.407501 98.03755) (end 350.307501 98.03755) (layer Edge.Cuts) (width 0.2))
   (gr_arc (start 302.801243 86.45) (end 302.801243 85.45) (angle -28.13752657) (layer Edge.Cuts) (width 0.2))
-  (gr_circle (center 312.5372 157.540591) (end 311.4372 157.540591) (layer Edge.Cuts) (width 0.2))
+  (gr_circle (center 312.5372 157.540591) (end 313.6372 157.540591) (layer Edge.Cuts) (width 0.2))
   (gr_arc (start 337.957501 79) (end 338.957501 79) (angle -90) (layer Edge.Cuts) (width 0.2))
   (gr_circle (center 170 88.95) (end 168.9 88.95) (layer Edge.Cuts) (width 0.2))
@@
   (segment (start 292.729568 161.949116) (end 296.324177 158.354507) (width 0.254) (layer B.Cu) (net 4))
   (segment (start 272.182754 161.949116) (end 292.729568 161.949116) (width 0.254) (layer B.Cu) (net 4))
-  (segment (start 345.809409 157.690591) (end 345.9645 157.690591) (width 0.254) (layer B.Cu) (net 4))
-  (segment (start 344 159.5) (end 345.809409 157.690591) (width 0.254) (layer B.Cu) (net 4))
-  (segment (start 297.8 159.5) (end 344 159.5) (width 0.254) (layer B.Cu) (net 4))
-  (segment (start 296.324177 158.354507) (end 296.654507 158.354507) (width 0.254) (layer B.Cu) (net 4))
-  (segment (start 296.654507 158.354507) (end 297.8 159.5) (width 0.254) (layer B.Cu) (net 4))
-  (segment (start 201.493355 173.358325) (end 201.841675 173.358325) (width 0.254) (layer B.Cu) (net 4))
-  (segment (start 201.841675 173.358325) (end 204.4 170.8) (width 0.254) (layer B.Cu) (net 4))
-  (via (at 204.4 170.8) (size 0.6) (drill 0.4) (layers F.Cu B.Cu) (net 4))
   (via (at 204.4 152.8) (size 0.6) (drill 0.4) (layers F.Cu B.Cu) (net 4))
-  (segment (start 204.4 170.8) (end 204.4 152.8) (width 0.254) (layer F.Cu) (net 4))
   (segment (start 204.4 140.146592) (end 204.4 152.375736) (width 0.254) (layer B.Cu) (net 4))
   (segment (start 207.75 136.796592) (end 204.4 140.146592) (width 0.254) (layer B.Cu) (net 4))
   (segment (start 207.75 135.653613) (end 207.75 136.796592) (width 0.254) (layer B.Cu) (net 4))
   (segment (start 204.4 152.375736) (end 204.4 152.8) (width 0.254) (layer B.Cu) (net 4))
-  (segment (start 245.984815 167.971689) (end 246.561401 167.395103) (width 0.254) (layer B.Cu) (net 4))
-  (segment (start 244.856504 169.1) (end 245.984815 167.971689) (width 0.254) (layer B.Cu) (net 4))
-  (segment (start 204.4 170.8) (end 206.1 169.1) (width 0.254) (layer B.Cu) (net 4))
-  (segment (start 206.1 169.1) (end 244.856504 169.1) (width 0.254) (layer B.Cu) (net 4))
+  (via (at 204.4 173.349999) (size 0.6) (drill 0.4) (layers F.Cu B.Cu) (net 4))
+  (segment (start 204.4 152.8) (end 204.4 173.349999) (width 0.254) (layer F.Cu) (net 4))
+  (segment (start 204.85 173.799999) (end 204.699999 173.649998) (width 0.254) (layer B.Cu) (net 4))
+  (segment (start 204.699999 173.649998) (end 204.4 173.349999) (width 0.254) (layer B.Cu) (net 4))
+  (segment (start 240.156505 173.799999) (end 204.85 173.799999) (width 0.254) (layer B.Cu) (net 4))
+  (segment (start 246.561401 167.395103) (end 240.156505 173.799999) (width 0.254) (layer B.Cu) (net 4))
+  (segment (start 204.391674 173.358325) (end 204.4 173.349999) (width 0.254) (layer B.Cu) (net 4))
+  (segment (start 201.493355 173.358325) (end 204.391674 173.358325) (width 0.254) (layer B.Cu) (net 4))
+  (segment (start 345.809409 157.690591) (end 345.9645 157.690591) (width 0.254) (layer B.Cu) (net 4))
+  (segment (start 342.5 161) (end 345.809409 157.690591) (width 0.254) (layer B.Cu) (net 4))
+  (segment (start 299.3 161) (end 342.5 161) (width 0.254) (layer B.Cu) (net 4))
+  (segment (start 296.324177 158.354507) (end 296.654507 158.354507) (width 0.254) (layer B.Cu) (net 4))
+  (segment (start 296.654507 158.354507) (end 299.3 161) (width 0.254) (layer B.Cu) (net 4))
   (segment (start 98.673751 115.586593) (end 98.673751 116.290593) (width 0.254) (layer B.Cu) (net 5))
   (segment (start 98.673751 113.998751) (end 98.673751 115.586593) (width 0.254) (layer B.Cu) (net 5))

Commit message: Update PCB
Parts:
- added K_SHIFT3: MX-1.25U, MX_Only:MXOnly-2.25U-NoLED, F.Cu at (334.0, 135.5)
- added K_SPC3: MX-2U, MX_Only:MXOnly-1.75U-NoLED, F.Cu at (163.6, 162.1)
- added K_SPC4: MX-1.75U, MX_Only:MXOnly-1U-NoLED, F.Cu at (230.6, 167.6)
- added K_WIN3: MX-1U, MX_Only:MXOnly-1.25U-NoLED, F.Cu at (191.5, 168.0)
- added K_WIN4: MX-1U, MX_Only:MXOnly-1.75U-NoLED, F.Cu at (256.2, 162.1)
- K_,1, K_.1, K_;1, K_A1, K_B1, K_B2, K_BSPC1, K_C1, K_D1, K_DEL1, K_E1, K_ESC1, K_F1, K_FN1, K_G1, K_H1, K_I1, K_J1, K_K1, K_L1, K_M1, K_N1, K_O1, K_P1, K_PGDN1, K_PGUP1, K_Q1, K_R1, K_S1, K_T1, K_U1, K_V1, K_W1, K_WIN1, K_WIN2, K_X1, K_Y1, K_Z1: footprint MX_Only:MXOnly-1U-Hotswap -> MX_Only:MXOnly-1U-NoLED
- K_ALT1, K_ALT2, K_CTRL1, K_CTRL2: footprint MX_Only:MXOnly-1.5U-Hotswap -> MX_Only:MXOnly-1.5U-NoLED
- K_ENTER1, K_SHIFT1, K_SPC2: footprint MX_Only:MXOnly-1.75U-Hotswap -> MX_Only:MXOnly-1.75U-NoLED
- K_SHIFT2, K_TAB1: footprint MX_Only:MXOnly-1.25U-Hotswap -> MX_Only:MXOnly-1.25U-NoLED
- K_SPC1: footprint MX_Only:MXOnly-2U-Hotswap-ReversedStabilizers -> MX_Only:MXOnly-2U-ReversedStabilizers-NoLED
- moved D39 6.00 mm to (333.0, 143.0)
- moved D40 6.00 mm to (336.0, 143.0)
Routing:
- net ROW3: track 303.7 -> 237.8 mm
- net Net-(D39-Pad2): track 6.03 -> 22.0 mm
- net COL3: track 156.0 -> 143.9 mm, vias 4 -> 0
- net Net-(D46-Pad2): track 6.11 -> 16.7 mm
- net Net-(D45-Pad2): track 6.09 -> 16.6 mm
- net COL4: track 111.2 -> 101.3 mm, vias 3 -> 0
- net COL2: track 150.5 -> 140.6 mm, vias 3 -> 0
- net COL6: track 95.1 -> 85.5 mm, vias 4 -> 0
- net COL5: track 113.8 -> 104.3 mm, vias 4 -> 0
- net COL1: track 195.5 -> 186.5 mm, vias 3 -> 0
- net COL12: track 155.2 -> 163.7 mm, vias 2 -> 0
- net COL9: track 119.0 -> 126.8 mm, vias 4 -> 0
- net Net-(D48-Pad2): track 6.05 -> 12.6 mm
- net Net-(D38-Pad2): track 6.05 -> 12.6 mm
- net Net-(D26-Pad2): track 6.05 -> 12.6 mm
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
Commit message: Add silk for different layouts
Other:
- board text added: "1.25u B"
- board text added: "1.25u E"
- board text added: "1.75u B"
- board text added: "1.75u C"
- board text added: "1.75u D"
- board text added: "1u A"
- board text added: "1u C"
- board text added: "1u D"
- board text added: "1u E"
- board text added: "2.25u F"
- board text added: "2u A"
Changed lines of the file:
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@@
   (general
     (thickness 1.6)
-    (drawings 190)
+    (drawings 201)
     (tracks 873)
     (zones 0)
@@
     )
   )
+  (gr_text "2.25u\nF" (at 334 127.95) (layer B.SilkS)
+    (effects (font (size 1 1) (thickness 0.2)) (justify mirror))
+  )
+  (gr_text "1u\nE" (at 348.8 141.1) (layer B.SilkS)
+    (effects (font (size 1 1) (thickness 0.2)) (justify mirror))
+  )
+  (gr_text "1.25u\nE" (at 325.3 141.15) (layer B.SilkS)
+    (effects (font (size 1 1) (thickness 0.2)) (justify mirror))
+  )
+  (gr_text "1.75u\nD" (at 257.75 167.45 12) (layer B.SilkS)
+    (effects (font (size 1 1) (thickness 0.2)) (justify mirror))
+  )
+  (gr_text "1u\nC" (at 264.45 165.95 12) (layer B.SilkS)
+    (effects (font (size 1 1) (thickness 0.2)) (justify mirror))
+  )
+  (gr_text "1u\nD" (at 232.1 172.9 12) (layer B.SilkS)
+    (effects (font (size 1 1) (thickness 0.2)) (justify mirror))
+  )
+  (gr_text "1.75u\nC" (at 239.05 171.4 12) (layer B.SilkS)
+    (effects (font (size 1 1) (thickness 0.2)) (justify mirror))
+  )
+  (gr_text "1.75u\nB" (at 161.15 167.15 -12) (layer B.SilkS)
+    (effects (font (size 1 1) (thickness 0.2)) (justify mirror))
+  )
+  (gr_text "2u\nA" (at 165.95 168.2 -12) (layer B.SilkS)
+    (effects (font (size 1 1) (thickness 0.2)) (justify mirror))
+  )
+  (gr_text "1u\nA" (at 193.35 174.05 -12) (layer B.SilkS)
+    (effects (font (size 1 1) (thickness 0.2)) (justify mirror))
+  )
+  (gr_text "1.25u\nB" (at 188.05 172.85 -12) (layer B.SilkS)
+    (effects (font (size 1 1) (thickness 0.2)) (justify mirror))
+  )
   (gr_circle (center 214.25 135.6) (end 214.55 135.6) (layer B.SilkS) (width 0.15))
