File: Vision.kicad_sch (KiCad schematic)
At the start: 145 parts, among them J1 Conn_ARM_JTAG_SWD_10, Q1 DTC123J, SW1 SW_Push, U1 MCP1700-3002E_SOT23, U2 STM32F072CBUx, U3 TPD4E05U06DQAR

Commit message: Use native Kicad USB-C footprint
Parts:
- USB1: footprint Type-C:HRO-TYPE-C-31-M-12-Assembly -> Connector_USB:USB_C_Receptacle_HRO_TYPE-C-31-M-12
Changed lines of the file:
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@@
       (effects (font (size 1.524 1.524)))
     )
-    (property "Footprint" "Type-C:HRO-TYPE-C-31-M-12-Assembly" (id 2) (at 41.91 163.83 0)
+    (property "Footprint" "Connector_USB:USB_C_Receptacle_HRO_TYPE-C-31-M-12" (id 2) (at 41.91 163.83 0)
       (effects (font (size 1.524 1.524)) hide)
     )
@@
     )
     (path "/00000000-0000-0000-0000-00005b361237"
-      (reference "USB1") (unit 1) (value "HRO-TYPE-C-31-M-12") (footprint "Type-C:HRO-TYPE-C-31-M-12-Assembly")
-    )
-  )
+      (reference "USB1") (unit 1) (value "HRO-TYPE-C-31-M-12") (footprint "Connector_USB:USB_C_Receptacle_HRO_TYPE-C-31-M-12")
+    )
+  )

Commit message: Final pre-proto changes
Parts:
- D50: LCSC C266723 -> C435473
- Q1: LCSC C111724 -> C968329
Changed lines of the file:
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@@
       (effects (font (size 1.27 1.27)) hide)
     )
-    (property "LCSC" "C266723" (id 4) (at 123.2916 167.1066 0)
+    (property "LCSC" "C435473" (id 4) (at 123.2916 167.1066 0)
       (effects (font (size 1.27 1.27)) hide)
     )
@@
       (effects (font (size 1.27 1.27)) (justify left) hide)
     )
-    (property "LCSC" "C111724" (id 4) (at 145.7452 242.0366 0)
-      (effects (font (size 1.27 1.27)) hide)
-    )
+    (property "LCSC" "C968329" (id 4) (at 145.7452 242.0366 0)
+      (effects (font (size 1.27 1.27)) hide)
+    )
